File: eagle/th_simple_ad.sch (EAGLE design)
At the start: 23 parts, among them IC1 TL071P, T1 2N3904

Commit message: file structure and one fixed value
Parts:
- removed OUT1: AUDIO-JACK, erthenvar:AUDIO-JACK
- added IC2: LM555N, adafruit:LM555N
- added OUT: AUDIO-JACK, erthenvar:AUDIO-JACK
- ATTACK, DECAY: value (none) -> 1M log
- D2: value 1N4148DO35-7 -> 1N4148DO35-10; device diode:1N4148DO35-7 -> diode:1N4148DO35-10
- R7: value 100k -> 10k
Connections:
- new net N$10: C7.1, IC2.CV
- net +12V: now also IC2.R, IC2.V+
- net GND: now also IC2.GND, OUT.RING; no longer OUT1.RING
- net N$11: now also IC2.DIS
- net N$3: now also OUT.TIP; no longer OUT1.TIP
- net N$5: now also IC2.THR
- net N$7: now also IC2.TR
- net N$8: now also IC2.Q
Other:
- moved on the sheet: C1, C2, C6, C7, D2, GATE, PWR1, R2, R5, R7, TRIG, U$1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

Commit message: vertical and cutout
Parts:
- C5: device rcl:C-US050-024X044 -> rcl:C-US075-032X103
Changed lines of the file:
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@@
 <grid distance="0.1" unitdist="inch" unit="inch" style="lines" multiple="1" display="no" altdistance="0.01" altunitdist="inch" altunit="inch"/>
 <layers>
-<layer number="1" name="Top" color="4" fill="1" visible="no" active="no"/>
-<layer number="16" name="Bottom" color="1" fill="1" visible="no" active="no"/>
-<layer number="17" name="Pads" color="2" fill="1" visible="no" active="no"/>
-<layer number="18" name="Vias" color="2" fill="1" visible="no" active="no"/>
-<layer number="19" name="Unrouted" color="6" fill="1" visible="no" active="no"/>
-<layer number="20" name="Dimension" color="15" fill="1" visible="no" active="no"/>
-<layer number="21" name="tPlace" color="7" fill="1" visible="no" active="no"/>
-<layer number="22" name="bPlace" color="7" fill="1" visible="no" active="no"/>
-<layer number="23" name="tOrigins" color="15" fill="1" visible="no" active="no"/>
-<layer number="24" name="bOrigins" color="15" fill="1" visible="no" active="no"/>
-<layer number="25" name="tNames" color="7" fill="1" visible="no" active="no"/>
-<layer number="26" name="bNames" color="7" fill="1" visible="no" active="no"/>
-<layer number="27" name="tValues" color="7" fill="1" visible="no" active="no"/>
-<layer number="28" name="bValues" color="7" fill="1" visible="no" active="no"/>
+<layer number="1" name="Top" color="4" fill="1" visible="yes" active="no"/>
+<layer number="16" name="Bottom" color="1" fill="1" visible="yes" active="no"/>
+<layer number="17" name="Pads" color="2" fill="1" visible="yes" active="no"/>
+<layer number="18" name="Vias" color="2" fill="1" visible="yes" active="no"/>
+<layer number="19" name="Unrouted" color="6" fill="1" visible="yes" active="no"/>
+<layer number="20" name="Dimension" color="15" fill="1" visible="yes" active="no"/>
+<layer number="21" name="tPlace" color="7" fill="1" visible="yes" active="no"/>
+<layer number="22" name="bPlace" color="7" fill="1" visible="yes" active="no"/>
+<layer number="23" name="tOrigins" color="15" fill="1" visible="yes" active="no"/>
+<layer number="24" name="bOrigins" color="15" fill="1" visible="yes" active="no"/>
+<layer number="25" name="tNames" color="7" fill="1" visible="yes" active="no"/>
+<layer number="26" name="bNames" color="7" fill="1" visible="yes" active="no"/>
+<layer number="27" name="tValues" color="7" fill="1" visible="yes" active="no"/>
+<layer number="28" name="bValues" color="7" fill="1" visible="yes" active="no"/>
 <layer number="29" name="tStop" color="7" fill="3" visible="no" active="no"/>
 <layer number="30" name="bStop" color="7" fill="6" visible="no" active="no"/>
@@
 <layer number="35" name="tGlue" color="7" fill="4" visible="no" active="no"/>
 <layer number="36" name="bGlue" color="7" fill="5" visible="no" active="no"/>
-<layer number="37" name="tTest" color="7" fill="1" visible="no" active="no"/>
-<layer number="38" name="bTest" color="7" fill="1" visible="no" active="no"/>
+<layer number="37" name="tTest" color="7" fill="1" visible="yes" active="no"/>
+<layer number="38" name="bTest" color="7" fill="1" visible="yes" active="no"/>
 <layer number="39" name="tKeepout" color="4" fill="11" visible="no" active="no"/>
 <layer number="40" name="bKeepout" color="1" fill="11" visible="no" active="no"/>
@@
 <layer number="44" name="Drills" color="7" fill="1" visible="no" active="no"/>
 <layer number="45" name="Holes" color="7" fill="1" visible="no" active="no"/>
-<layer number="46" name="Milling" color="3" fill="1" visible="no" active="no"/>
-<layer number="47" name="Measures" color="7" fill="1" visible="no" active="no"/>
-<layer number="48" name="Document" color="7" fill="1" visible="no" active="no"/>
-<layer number="49" name="Reference" color="7" fill="1" visible="no" active="no"/>
-<layer number="50" name="dxf" color="7" fill="1" visible="no" active="no"/>
-<layer number="51" name="tDocu" color="7" fill="1" visible="no" active="no"/>
-<layer number="52" name="bDocu" color="7" fill="1" visible="no" active="no"/>
-<layer number="53" name="tGND_GNDA" color="7" fill="9" visible="no" active="no"/>
-<layer number="54" name="bGND_GNDA" color="1" fill="9" visible="no" active="no"/>
-<layer number="56" name="wert" color="7" fill="1" visible="no" active="no"/>
-<layer number="57" name="tCAD" color="7" fill="1" visible="no" active="no"/>
-<layer number="59" name="tCarbon" color="7" fill="1" visible="no" active="no"/>
-<layer number="60" name="bCarbon" color="7" fill="1" visible="no" active="no"/>
+<layer number="46" name="Milling" color="3" fill="1" visible="yes" active="no"/>
+<layer number="47" name="Measures" color="7" fill="1" visible="yes" active="no"/>
+<layer number="48" name="Document" color="7" fill="1" visible="yes" active="no"/>
+<layer number="49" name="Reference" color="7" fill="1" visible="yes" active="no"/>
+<layer number="50" name="dxf" color="7" fill="1" visible="yes" active="no"/>
+<layer number="51" name="tDocu" color="7" fill="1" visible="yes" active="no"/>
+<layer number="52" name="bDocu" color="7" fill="1" visible="yes" active="no"/>
+<layer number="53" name="tGND_GNDA" color="7" fill="9" visible="yes" active="no"/>
+<layer number="54" name="bGND_GNDA" color="1" fill="9" visible="yes" active="no"/>
+<layer number="56" name="wert" color="7" fill="1" visible="yes" active="no"/>
+<layer number="57" name="tCAD" color="7" fill="1" visible="yes" active="no"/>
+<layer number="59" name="tCarbon" color="7" fill="1" visible="yes" active="no"/>
+<layer number="60" name="bCarbon" color="7" fill="1" visible="yes" active="no"/>
 <layer number="90" name="Modules" color="5" fill="1" visible="yes" active="yes"/>
 <layer number="91" name="Nets" color="2" fill="1" visible="yes" active="yes"/>
@@
 <part name="GND6" library="supply1" deviceset="GND" device=""/>
 <part name="TRIG" library="erthenvar" deviceset="AUDIO-JACK" device=""/>
-<part name="C5" library="rcl" deviceset="C-US" device="050-024X044" value="100p"/>
+<part name="C5" library="rcl" deviceset="C-US" device="075-032X103" value="100p"/>
 <part name="R6" library="rcl" deviceset="R-US_" device="0207/10" value="100k"/>
 <part name="D1" library="diode" deviceset="1N4148" device="DO35-7" value="1N4148DO35-7"/>

Commit message: verified
Parts:
- C5: device rcl:C-US075-032X103 -> rcl:C-US050-024X044
- D2: value 1N4148DO35-10 -> 1N4148DO35-7; device diode:1N4148DO35-10 -> diode:1N4148DO35-7
Changed lines of the file:
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@@
 <part name="GND6" library="supply1" deviceset="GND" device=""/>
 <part name="TRIG" library="erthenvar" deviceset="AUDIO-JACK" device=""/>
-<part name="C5" library="rcl" deviceset="C-US" device="075-032X103" value="100p"/>
+<part name="C5" library="rcl" deviceset="C-US" device="050-024X044" value="100p"/>
 <part name="R6" library="rcl" deviceset="R-US_" device="0207/10" value="100k"/>
 <part name="D1" library="diode" deviceset="1N4148" device="DO35-7" value="1N4148DO35-7"/>
@@
 <part name="C7" library="rcl" deviceset="C-US" device="050-024X044" value="10n"/>
 <part name="GND11" library="supply1" deviceset="GND" device=""/>
-<part name="D2" library="diode" deviceset="1N4148" device="DO35-10" value="1N4148DO35-10"/>
+<part name="D2" library="diode" deviceset="1N4148" device="DO35-7" value="1N4148DO35-7"/>
 <part name="DECAY" library="pot" deviceset="3RP/1610N" device="" value="1M log"/>
 <part name="ATTACK" library="pot" deviceset="3RP/1610N" device="" value="1M log"/>
